Commit message: making the module flexible

File: src/mybot_description/parts/cameras.xacro (robot description, xacro)
@@ -2,13 +2,28 @@
 <robot name="myrobot" xmlns:xacro="http://www.ros.org/wiki/xacro">
  <xacro:property name="base_line" value="chassis"/>
- <xacro:property name="cameraWeight" value="0.01"/>
+ <xacro:property name="cameraWidth" value="0.01"/>
  <xacro:property name="cameraLength" value="0.09"/>
  <xacro:property name="cameraHight" value="0.05"/>
  <xacro:property name="cameraMass" value="0.1"/>
+  <xacro:property name="camera_f_x" value="0"/>
+  <xacro:property name="camera_f_y" value="0"/>
+  <xacro:property name="camera_f_z" value="0"/>
+  <xacro:property name="camera_r_x" value="0"/>
+  <xacro:property name="camera_r_y" value="0"/>
+  <xacro:property name="camera_r_z" value="0"/>
+  <xacro:property name="camera_l_x" value="0"/>
+  <xacro:property name="camera_l_y" value="0"/>
+  <xacro:property name="camera_l_z" value="0"/>
+  <xacro:property name="camera_b_x" value="0"/>
+  <xacro:property name="camera_b_y" value="0"/>
+  <xacro:property name="camera_b_z" value="0"/>
+  <xacro:property name="orig_x" value="${chassis_x + bar_x}"/>
+  <xacro:property name="orig_y" value="${chassis_y + bar_y}"/>
+  <xacro:property name="orig_z" value="${chassis_z +chassis_H/2 + bar_H + bar_z - cameraHight/2 }"/>
     <link name="camera_front">
     <collision>
       <origin xyz="0 0 0" rpy="0 0 0"/>
       <geometry>
-        <box size="${cameraWeight} ${cameraLength} ${cameraHight}"/>
+        <box size="${cameraWidth} ${cameraLength} ${cameraHight}"/>
       </geometry>
     </collision>
@@ -16,5 +31,5 @@
       <origin xyz="0 0 0" rpy="0 0 0"/>
       <geometry>
-        <box size="${cameraWeight} ${cameraLength} ${cameraHight}"/>
+        <box size="${cameraWidth} ${cameraLength} ${cameraHight}"/>
       </geometry>
       <material name="green"/>
@@ -23,5 +38,5 @@
       <mass value="${cameraMass}" />
       <origin xyz="0 0 0" rpy="0 0 0"/>
-      <box_inertia m="${cameraMass}" x="${cameraWeight}" y="${cameraLength}" z="${cameraHight}" />
+      <box_inertia m="${cameraMass}" x="${cameraWidth}" y="${cameraLength}" z="${cameraHight}" />
       <inertia ixx="1e-6" ixy="0" ixz="0" iyy="1e-6" iyz="0" izz="1e-6" />
     </inertial>
@@ -29,5 +44,5 @@
   <joint name="camera_front_joint" type="fixed">
     <axis xyz="0 1 0" />
-    <origin xyz=".055 0 0.2" rpy="0 0 0"/>
+    <origin xyz="${orig_x + bar_L/2 + cameraWidth/2 + camera_f_x} ${orig_y  +  camera_f_y}  ${orig_z + camera_f_z}" rpy="0 0 0"/>
     <parent link="${base_line}"/>
     <child link="camera_front"/>
@@ -37,5 +52,5 @@
       <origin xyz="0 0 0" rpy="0 0 0"/>
       <geometry>
-        <box size="${cameraWeight} ${cameraLength} ${cameraHight}"/>
+        <box size="${cameraWidth} ${cameraLength} ${cameraHight}"/>
       </geometry>
     </collision>
@@ -43,5 +58,5 @@
       <origin xyz="0 0 0" rpy="0 0 0"/>
       <geometry>
-        <box size="${cameraWeight} ${cameraLength} ${cameraHight}"/>
+        <box size="${cameraWidth} ${cameraLength} ${cameraHight}"/>
       </geometry>
       <material name="green"/>
@@ -50,5 +65,5 @@
       <mass value="${cameraMass}" />
       <origin xyz="0 0 0" rpy="0 0 0"/>
-      <box_inertia m="${cameraMass}" x="${cameraWeight}" y="${cameraLength}" z="${cameraHight}" />
+      <box_inertia m="${cameraMass}" x="${cameraWidth}" y="${cameraLength}" z="${cameraHight}" />
       <inertia ixx="1e-6" ixy="0" ixz="0" iyy="1e-6" iyz="0" izz="1e-6" />
     </inertial>
@@ -56,5 +71,6 @@
   <joint name="camera_back_joint" type="fixed">
     <axis xyz="0 0 0" />
-    <origin xyz="-.055 0 0.2" rpy="0 0 3.14"/>
+    <origin xyz="${orig_x - bar_L/2 - cameraWidth/2 + camera_b_x} ${orig_y+ camera_b_y}  ${orig_z + camera_b_z}"
+      rpy="0 0 3.14"/>
     <parent link="${base_line}"/>
     <child link="camera_back"/>
@@ -64,5 +80,5 @@
       <origin xyz="0 0 0" rpy="0 0 0"/>
       <geometry>
-        <box size="${cameraWeight} ${cameraLength} ${cameraHight}"/>
+        <box size="${cameraWidth} ${cameraLength} ${cameraHight}"/>
       </geometry>
     </collision>
@@ -70,5 +86,5 @@
       <origin xyz="0 0 0" rpy="0 0 0"/>
       <geometry>
-        <box size="${cameraWeight} ${cameraLength} ${cameraHight}"/>
+        <box size="${cameraWidth} ${cameraLength} ${cameraHight}"/>
       </geometry>
       <material name="green"/>
@@ -77,5 +93,5 @@
       <mass value="${cameraMass}" />
       <origin xyz="0 0 0" rpy="0 0 0"/>
-      <box_inertia m="${cameraMass}" x="${cameraWeight}" y="${cameraLength}" z="${cameraHight}" />
+      <box_inertia m="${cameraMass}" x="${cameraWidth}" y="${cameraLength}" z="${cameraHight}" />
       <inertia ixx="1e-6" ixy="0" ixz="0" iyy="1e-6" iyz="0" izz="1e-6" />
     </inertial>
@@ -83,5 +99,6 @@
   <joint name="camera_right_joint" type="fixed">
     <axis xyz="0 0 0" />
-    <origin xyz="0 -0.055 0.2" rpy="0 0 -1.57"/>
+    <origin xyz="${orig_x + camera_r_x} ${orig_y - cameraWidth/2 - bar_W/2 + camera_r_y }  ${orig_z + camera_r_z}"
+    rpy="0 0 -1.57"/>
     <parent link="${base_line}"/>
     <child link="camera_right"/>
@@ -91,5 +108,5 @@
       <origin xyz="0 0 0" rpy="0 0 0"/>
       <geometry>
-        <box size="${cameraWeight} ${cameraLength} ${cameraHight}"/>
+        <box size="${cameraWidth} ${cameraLength} ${cameraHight}"/>
       </geometry>
     </collision>
@@ -97,5 +114,5 @@
       <origin xyz="0 0 0" rpy="0 0 0"/>
       <geometry>
-        <box size="${cameraWeight} ${cameraLength} ${cameraHight}"/>
+        <box size="${cameraWidth} ${cameraLength} ${cameraHight}"/>
       </geometry>
       <material name="green"/>
@@ -104,5 +121,5 @@
       <mass value="${cameraMass}" />
       <origin xyz="0 0 0" rpy="0 0 0"/>
-      <box_inertia m="${cameraMass}" x="${cameraWeight}" y="${cameraLength}" z="${cameraHight}" />
+      <box_inertia m="${cameraMass}" x="${cameraWidth}" y="${cameraLength}" z="${cameraHight}" />
       <inertia ixx="1e-6" ixy="0" ixz="0" iyy="1e-6" iyz="0" izz="1e-6" />
     </inertial>
@@ -110,5 +127,6 @@
   <joint name="camera_left_joint" type="fixed">
     <axis xyz="0 0 0" />
-    <origin xyz="0 0.055 0.2" rpy="0 0 1.57"/>
+    <origin xyz="${chassis_x + bar_x + camera_l_x} ${orig_y + cameraWidth/2 + bar_W/2 + camera_l_y}  ${orig_z + camera_l_z}"
+    rpy="0 0 1.57"/>
     <parent link="${base_line}"/>
     <child link="camera_left"/>

File: src/mybot_description/parts/lidar_2d.xacro (robot description, xacro)
@@ -3,5 +3,5 @@
   <joint name="hokuyo_joint" type="fixed">
     <axis xyz="0 1 0" />
-    <origin xyz=".15 0 .1" rpy="0 0 0"/>
+    <origin xyz="${chassis_x + chassis_L/2 + lidar_x} ${chassis_y + lidar_y} ${chassis_z + chassis_H/2 + lidar_z}" rpy="0 0 0"/>
     <parent link="chassis"/>
     <child link="hokuyo"/>

File: src/mybot_description/parts/velodyne.xacro (robot description, xacro)
@@ -4,6 +4,12 @@
   <xacro:property name="gpu" value="$(arg gpu)" />
   <xacro:include filename="$(find velodyne_description)/urdf/VLP-16.urdf.xacro"/>
+ <xacro:property name="velodyne_x" value="0"/>
+ <xacro:property name="velodyne_y" value="0.2"/>
+ <xacro:property name="velodyne_z" value="0."/>
+   <xacro:property name="orig_x" value="${chassis_x + bar_x}"/>
+  <xacro:property name="orig_y" value="${chassis_y + bar_y}"/>
+  <xacro:property name="orig_z" value="${chassis_z + chassis_H/2 + bar_H + bar_z  }"/>
  <VLP-16 parent="chassis" name="velodyne" topic="/velodyne_points" hz="10" samples="440" gpu="${gpu}">
-    <origin xyz="0 0 0.25" rpy="0 0 0" />
+    <origin xyz="${orig_x} ${orig_y} ${orig_z + velodyne_z}" rpy="0 0 0" />
   </VLP-16>
 </robot>

File: src/mybot_description/parts/wheels.xacro (robot description, xacro)
@@ -5,5 +5,5 @@
       <origin xyz="0 0 0" rpy="0 1.5707 1.5707"/>
       <geometry>
-        <cylinder radius="0.1" length="0.05"/>
+        <cylinder radius="${wheel_R}" length="${wheel_L}"/>
       </geometry>
     </collision>
@@ -11,10 +11,10 @@
       <origin xyz="0 0 0" rpy="0 1.5707 1.5707"/>
       <geometry>
-        <cylinder radius="0.1" length="0.05"/>
+        <cylinder radius="${wheel_R}" length="${wheel_L}"/>
       </geometry>
     </visual>
     <inertial>
       <origin xyz="0 0 0" rpy="0 1.5707 1.5707"/>
-      <mass value="5"/>
+      <mass value="${wheels_mass}"/>
       <inertia
         ixx=".1" ixy="0.0" ixz="0.0"
@@ -27,5 +27,5 @@
       <origin xyz="0 0 0" rpy="0 1.5707 1.5707"/>
       <geometry>
-        <cylinder radius="0.1" length="0.05"/>
+        <cylinder radius="${wheel_R}" length="${wheel_L}"/>
       </geometry>
     </collision>
@@ -33,10 +33,10 @@
       <origin xyz="0 0 0" rpy="0 1.5707 1.5707"/>
       <geometry>
-        <cylinder radius="0.1" length="0.05"/>
+        <cylinder radius="${wheel_R}" length="${wheel_L}"/>
       </geometry>
     </visual>
     <inertial>
       <origin xyz="0 0 0" rpy="0 1.5707 1.5707"/>
-      <mass value="5"/>
+      <mass value="${wheels_mass}"/>
       <inertia
         ixx=".1" ixy="0.0" ixz="0.0"
@@ -49,5 +49,5 @@
       <origin xyz="0 0 0" rpy="0 1.5707 1.5707"/>
       <geometry>
-        <cylinder radius="0.1" length="0.05"/>
+        <cylinder radius="${wheel_R}" length="${wheel_L}"/>
       </geometry>
     </collision>
@@ -55,10 +55,10 @@
       <origin xyz="0 0 0" rpy="0 1.5707 1.5707"/>
       <geometry>
-        <cylinder radius="0.1" length="0.05"/>
+        <cylinder  radius="${wheel_R}" length="${wheel_L}"/>
       </geometry>
     </visual>
     <inertial>
       <origin xyz="0 0 0" rpy="0 1.5707 1.5707"/>
-      <mass value="5"/>
+      <mass value="${wheels_mass}"/>
       <inertia
         ixx=".1" ixy="0.0" ixz="0.0"
@@ -67,9 +67,9 @@
     </inertial>
   </link>
-    <link name="right_wheel_1">
+  <link name="right_wheel_1">
     <collision name="collision">
       <origin xyz="0 0 0" rpy="0 1.5707 1.5707"/>
       <geometry>
-        <cylinder radius="0.1" length="0.05"/>
+        <cylinder  radius="${wheel_R}" length="${wheel_L}"/>
       </geometry>
     </collision>
@@ -77,10 +77,10 @@
       <origin xyz="0 0 0" rpy="0 1.5707 1.5707"/>
       <geometry>
-        <cylinder radius="0.1" length="0.05"/>
+        <cylinder  radius="${wheel_R}" length="${wheel_L}"/>
       </geometry>
     </visual>
     <inertial>
       <origin xyz="0 0 0" rpy="0 1.5707 1.5707"/>
-      <mass value="5"/>
+      <mass value="${wheels_mass}"/>
       <inertia
         ixx=".1" ixy="0.0" ixz="0.0"
@@ -89,6 +89,6 @@
     </inertial>
   </link>
-    <joint type="continuous" name="left_wheel_hinge">
-    <origin xyz="0.11 0.15 0" rpy="0 0 0"/>
+  <joint type="continuous" name="left_wheel_hinge">
+    <origin xyz="${(chassis_x + chassis_L/2 - wheel_R)} ${chassis_y + (chassis_W/2 + wheel_L/2 + wheels_offset )} ${chassis_z - chassis_H/2}" rpy="0 0 0"/>
     <child link="left_wheel"/>
     <parent link="chassis"/>
@@ -98,5 +98,5 @@
   </joint>
   <joint type="continuous" name="left_wheel_hinge_1">
-    <origin xyz="-0.11 0.15 0" rpy="0 0 0"/>
+    <origin xyz="${chassis_x - (chassis_L/2 - wheel_R)} ${chassis_y + (chassis_W/2 + wheel_L/2 + wheels_offset)} ${chassis_z - chassis_H/2}" rpy="0 0 0"/>
     <child link="left_wheel_1"/>
     <parent link="chassis"/>
@@ -106,5 +106,5 @@
   </joint>
   <joint type="continuous" name="right_wheel_hinge">
-    <origin xyz="0.11 -0.15 0" rpy="0 0 0"/>
+    <origin xyz="${(chassis_x + chassis_L/2 - wheel_R)} ${chassis_y - (chassis_W/2 + wheel_L/2 + wheels_offset)} ${chassis_z - chassis_H/2}" rpy="0 0 0"/>
     <child link="right_wheel"/>
     <parent link="chassis"/>
@@ -114,5 +114,5 @@
   </joint>
   <joint type="continuous" name="right_wheel_hinge_1">
-    <origin xyz="-0.11 -0.15 0" rpy="0 0 0"/>
+    <origin xyz="${chassis_x - (chassis_L/2 - wheel_R)} ${chassis_y - (chassis_W/2 + wheel_L/2 + wheels_offset)} ${chassis_z - chassis_H/2}" rpy="0 0 0"/>
     <child link="right_wheel_1"/>
     <parent link="chassis"/>

File: src/mybot_description/urdf/mybot.xacro (robot description, xacro)
@@ -1,4 +1,5 @@
 <?xml version='1.0'?>
 <robot name="myrobot" xmlns:xacro="http://www.ros.org/wiki/xacro">
+  <xacro:include filename="$(find mybot_description)/urdf/parameter.xacro" />
   <xacro:include filename="$(find mybot_description)/urdf/mybot.gazebo" />
   <xacro:include filename="$(find mybot_description)/urdf/materials.xacro" />
@@ -26,11 +27,11 @@
     <collision name='collision'>
       <geometry>
-        <box size=".4 .2 .1"/>
+        <box size="${chassis_L}  ${chassis_W}  ${chassis_H}"/>
       </geometry>
     </collision>
     <visual name='chassis_visual'>
-      <origin xyz="0 0 0" rpy=" 0 0 0"/>
+      <origin xyz="${chassis_x}  ${chassis_y} ${chassis_z}" rpy=" 0 0 0"/>
       <geometry>
-        <box size=".4 .2 .1"/>
+        <box size="${chassis_L}  ${chassis_W}  ${chassis_H}"/>
       </geometry>
     </visual>
@@ -49,16 +50,16 @@
     <collision name='collision'>
       <geometry>
-        <box size=".1 .1 .4"/>
+        <box size="${bar_L}  ${bar_W}  ${bar_H}"/>
       </geometry>
     </collision>
     <visual name='bar_visual'>
-      <origin xyz="0 0 0" rpy=" 0 0 0"/>
+      <origin xyz="0 0 ${bar_H/2}" rpy=" 0 0 0"/>
       <geometry>
-        <box size=".1 .1 .2"/>
+        <box size="${bar_L}  ${bar_W}  ${bar_H}"/>
       </geometry>
     </visual>
   </link>
   <joint name="bar_joint" type="fixed">
-    <origin xyz="0 0 0.15" rpy="0 0 0"/>
+    <origin xyz="${chassis_x + bar_x} ${chassis_y + bar_y} ${chassis_z + chassis_H/2 + bar_z}" rpy="0 0 0"/>
     <parent link="chassis"/>
     <child link="bar"/>
