Commit message: adding mini_jaguar_pkg

File: src/mybot_description/urdf/mybot.xacro (robot description, xacro)
@@ -4,7 +4,7 @@
   <xacro:include filename="$(find mybot_description)/urdf/mybot.gazebo" />
   <xacro:include filename="$(find mybot_description)/urdf/materials.xacro" />
-  <xacro:include filename="$(find mybot_description)/parts/velodyne.xacro" />
+  <!-- <xacro:include filename="$(find mybot_description)/parts/velodyne.xacro" /> -->
   <xacro:include filename="$(find mybot_description)/parts/wheels.xacro" />
-  <xacro:include filename="$(find mybot_description)/parts/cameras.xacro" />
+  <!-- <xacro:include filename="$(find mybot_description)/parts/cameras.xacro" />  -->
   <xacro:include filename="$(find mybot_description)/parts/lidar_2d.xacro" />
   <link name="base_link">
@@ -17,5 +17,5 @@
     <pose>0 0 0.1 0 0 0</pose>
     <inertial>
-      <mass value="15.0"/>
+      <mass value="${chassis_mass}"/>
       <origin xyz="0.0 0 0.1" rpy=" 0 0 0"/>
       <inertia

File: src/mybot_description/urdf/parameter.xacro (robot description, xacro)
@@ -4,7 +4,8 @@
 <xacro:property name="chassis_y" value="0" />
 <xacro:property name="chassis_z" value="0" />
-<xacro:property name="chassis_L" value="0.4" />
-<xacro:property name="chassis_W" value="0.2" />
-<xacro:property name="chassis_H" value="0.1" />
+<xacro:property name="chassis_L" value="0.6858" />
+<xacro:property name="chassis_W" value="0.4064" />
+<xacro:property name="chassis_H" value="0.1524" />
+<xacro:property name="chassis_mass" value="10" />
 <xacro:property name="bar_L" value="0.1" />
 <xacro:property name="bar_W" value="0.1" />
@@ -13,8 +14,9 @@
 <xacro:property name="bar_y" value="0" />
 <xacro:property name="bar_z" value="0" />
-<xacro:property name="wheel_R" value="0.05" />
-<xacro:property name="wheel_L" value="0.03" />
+<xacro:property name="wheel_R" value="0.15" />
+<xacro:property name="wheel_L" value="0.05" />
+<!-- off set the wheel from the chassis -->
 <xacro:property name="wheels_offset" value="0.01" />
-<xacro:property name="wheels_mass" value="5" />
+<xacro:property name="wheels_mass" value="2" />
 <xacro:property name="lidar_x" value="-0.025" />
 <xacro:property name="lidar_y" value="0" />
