Commit message: reorganizing the package adding arm controller

File: src/mini_jaguar_pkg/parts/arm.xacro (robot description, xacro)
@@ -2,14 +2,13 @@
 <robot xmlns:xacro="http://www.ros.org/wiki/xacro">
     <xacro:property name="arm_mass" value="2" />
-              <!-- origin_rpy="0 0 0" origin_xyz="0.2 0 0.05" -->
+   <xacro:property name="joints_friction" value="5" />
 <!-- Base Arm -->
-  <m_joint_1 name="${link_00_name}__${link_01_name}" type="revolute"
+  <m_joint_2 name="${link_00_name}__${link_01_name}" type="revolute"
            axis_xyz="0 0 1"
-           frict="0.5"
+           frict="${joints_friction}"
            damp="0.2"
            origin_rpy="0 0 0" origin_xyz="${ chassis_L/2 + ArmBase_x - 0.13} ${ ArmBase_y} ${chassis_H + ArmBase_z - 0.028}"
            parent="${link_00_name}" child="${link_01_name}"
-           limit_e="0" limit_l="0" limit_u="0" limit_v="0" />
-                   <!-- limit_e="0" limit_l="-3.14" limit_u="3.14" limit_v="0.5" />    -->
+          limit_e="0" limit_l="-2.0" limit_u="2.0" limit_v="0.5" />
   <m_link_mesh name="${link_01_name}"
               origin_rpy="0 0 0" origin_xyz="0 0 0"
@@ -21,12 +20,11 @@
               meshscale="0.0003 0.0003 0.0003" />
 <!--  Arm 1 -->
-  <m_joint_1 name="${link_01_name}__${link_06_name}" type="revolute"
+  <m_joint_2 name="${link_01_name}__${link_06_name}" type="revolute"
            axis_xyz="0 1 0"
-           frict="0.5"
+           frict="${joints_friction}"
            damp="0.2"
            origin_rpy="0 3.14 0" origin_xyz="0 0 0.13"
            parent="${link_01_name}" child="${link_06_name}"
            limit_e="1000" limit_l="0" limit_u="2.5" limit_v="0.5" />
-                <!-- limit_e="0" limit_l="0" limit_u="0" limit_v="0" />     -->
   <m_link_mesh name="${link_06_name}"
               origin_rpy="0 0 0" origin_xyz="0 -0.0145 -0.0145"
@@ -38,12 +36,11 @@
               meshscale="0.004 0.0029 0.003" />
 <!--  Arm 2 -->
-  <m_joint_1 name="${link_06_name}__${link_07_name}" type="revolute"
+  <m_joint_2 name="${link_06_name}__${link_07_name}" type="revolute"
            axis_xyz="0 1 0"
-           frict="0.5"
+           frict="${joints_friction}"
            damp="0.2"
-           origin_rpy="3.14 3.14 0" origin_xyz="0.44 0 -0.015"
+           origin_rpy="3.14 3.09 0" origin_xyz="0.44 0 -0.015"
            parent="${link_06_name}" child="${link_07_name}"
            limit_e="1000" limit_l="0.00" limit_u="3.14" limit_v="0.5" />
-                   <!-- limit_e="0" limit_l="0" limit_u="0" limit_v="0" />   -->
   <m_link_mesh name="${link_07_name}"
               origin_rpy="0 0 0" origin_xyz="0 -0.0145 -0.03"
@@ -55,12 +52,11 @@
               meshscale="0.004 0.0029 0.003" />
 <!--  Arm 3 -->
-  <m_joint_1 name="${link_07_name}__${link_08_name}" type="revolute"
+  <m_joint_2 name="${link_07_name}__${link_08_name}" type="revolute"
            axis_xyz="0 1 0"
-            frict="0.5"
+            frict="${joints_friction}"
            damp="0.2"
-           origin_rpy="0 0 0" origin_xyz="0.43 0.025 -0.0145"
+           origin_rpy="0 0 0" origin_xyz="0.43 0.035 -0.015"
            parent="${link_07_name}" child="${link_08_name}"
-             limit_e="0" limit_l="0" limit_u="0" limit_v="0" />
-              <!-- limit_e="1000" limit_l="-3.14" limit_u="3.14" limit_v="0.5" /> -->
+           limit_e="1000" limit_l="-3.14" limit_u="3.14" limit_v="0.5" />
   <m_link_mesh name="${link_08_name}"
               origin_rpy="0 0 0" origin_xyz="-0.15  -0.0145 -0.0145"
@@ -72,12 +68,11 @@
               meshscale="0.0025 0.0029 0.003" />
 <!--  gripper base  3 -->
-  <m_joint_1 name="${link_08_name}__${link_09_name}" type="revolute"
+  <m_joint_2 name="${link_08_name}__${link_09_name}" type="revolute"
            axis_xyz="0 0 1"
-           frict="0.5"
+           frict="${joints_friction}"
            damp="0.2"
            origin_rpy="0 1.57079 0" origin_xyz="0.13 0 0"
            parent="${link_08_name}" child="${link_09_name}"
            limit_e="1000" limit_l="-3.14" limit_u="3.14" limit_v="0.5" />
- <!-- limit_e="0" limit_l="0" limit_u="0" limit_v="0" /> -->
   <m_link_cylinder name="${link_09_name}"
               origin_rpy="0 0 0" origin_xyz="0 0 0"
@@ -88,7 +83,7 @@
               radius='.015' length='0.01'/>
 <!--  gripper arm  10 -->
-  <m_joint_1 name="${link_09_name}__${link_10_name}" type="revolute"
+  <m_joint_2 name="${link_09_name}__${link_10_name}" type="revolute"
            axis_xyz="1 0 0"
-           frict="0.5"
+           frict="${joints_friction}"
            damp="0.2"
            origin_rpy="0 0 0" origin_xyz="0 0.018 0.01"
@@ -103,7 +98,7 @@
               size='0.02 0.005 0.05'/>
 <!--  gripper arm  11 -->
-  <m_joint_1 name="${link_09_name}__${link_11_name}" type="revolute"
+  <m_joint_2 name="${link_09_name}__${link_11_name}" type="revolute"
            axis_xyz="1 0 0"
-           frict="0.5"
+           frict="${joints_friction}"
            damp="0.2"
            origin_rpy="0 0 3.14" origin_xyz="0 -0.018 0.01"

File: src/mini_jaguar_pkg/parts/cameras.xacro (robot description, xacro)
@@ -1,4 +1,5 @@
 <?xml version='1.0'?>
 <robot name="myrobot" xmlns:xacro="http://www.ros.org/wiki/xacro">
+  <xacro:include filename="$(find mini_jaguar_pkg)/gazebo_plugin/camera.gazebo" />
  <xacro:property name="base_line" value="chassis"/>
  <xacro:property name="cameraWidth" value="0.01"/>

File: src/mini_jaguar_pkg/parts/lidar_2d.xacro (robot description, xacro)
@@ -1,4 +1,5 @@
 <?xml version='1.0'?>
 <robot name="myrobot" xmlns:xacro="http://www.ros.org/wiki/xacro">
+  <xacro:include filename="$(find mini_jaguar_pkg)/gazebo_plugin/lidar.gazebo" />
   <joint name="hokuyo_joint" type="fixed">
     <axis xyz="0 1 0" />

File: src/mini_jaguar_pkg/parts/wheels.xacro (robot description, xacro)
@@ -1,4 +1,5 @@
 <?xml version="1.0" ?>
 <robot xmlns:xacro="http://www.ros.org/wiki/xacro">
+  <xacro:include filename="$(find mini_jaguar_pkg)/gazebo_plugin/wheels.gazebo" />
 <!-- <xacro:property name="wheels_mass" value="2" /> -->
    <m_joint name="${link_00_name}__${link_02_name}" type="continuous"

File: src/mini_jaguar_pkg/urdf/links_joints.xacro (robot description, xacro)
@@ -36,4 +36,24 @@
       <actuator name="motor_${name}">
         <hardwareInterface>hardware_interface/EffortJointInterface</hardwareInterface>
+        <mechanicalReduction>1</mechanicalReduction>
+      </actuator>
+    </transmission>
+  </xacro:macro>
+    <xacro:macro name="m_joint_2" params="name type axis_xyz origin_rpy origin_xyz damp frict parent child limit_e limit_l limit_u limit_v">
+    <joint name="${name}" type="${type}">
+      <axis xyz="${axis_xyz}" />
+      <dynamics damping="${damp}" friction="${frict}"/>
+      <limit effort="${limit_e}" lower="${limit_l}" upper="${limit_u}" velocity="${limit_v}" />
+      <origin rpy="${origin_rpy}" xyz="${origin_xyz}" />
+      <parent link="${parent}" />
+      <child link="${child}" />
+    </joint>
+    <transmission name="trans_${name}">
+      <type>transmission_interface/SimpleTransmission</type>
+      <joint name="${name}">
+        <hardwareInterface>hardware_interface/PositionJointInterface</hardwareInterface>
+      </joint>
+      <actuator name="motor_${name}">
+        <hardwareInterface>hardware_interface/PositionJointInterface</hardwareInterface>
         <mechanicalReduction>1</mechanicalReduction>
       </actuator>

File: src/mini_jaguar_pkg/urdf/mini.xacro (robot description, xacro)
@@ -6,8 +6,8 @@
    <xacro:include filename="$(find mini_jaguar_pkg)/parts/wheels.xacro" />
    <xacro:include filename="$(find mini_jaguar_pkg)/parts/lidar_2d.xacro" />
-   <xacro:include filename="$(find mini_jaguar_pkg)/parts/velodyne.xacro" />
+   <!-- <xacro:include filename="$(find mini_jaguar_pkg)/parts/velodyne.xacro" /> -->
    <xacro:include filename="$(find mini_jaguar_pkg)/parts/arm.xacro" />
    <!-- <xacro:include filename="$(find mini_jaguar_pkg)/parts/fins.xacro" />  -->
-  <xacro:include filename="$(find mini_jaguar_pkg)/urdf/mini.gazebo" />
+  <xacro:include filename="$(find mini_jaguar_pkg)/gazebo_plugin/genral.gazebo" />
   <!-- END - Include -->
   <link name="${dummy_link}">

File: src/mini_jaguar_pkg/urdf/robot_parameters.xacro (robot description, xacro)
@@ -24,6 +24,6 @@
 <xacro:property name="off_The_Ground" value="0.00" />
 <xacro:property name="chassis_L" value="${0.6858  }" />
-<xacro:property name="chassis_W" value="${0.4064 }" />
-<xacro:property name="chassis_H" value="0.1524" />
+<xacro:property name="chassis_W" value="${0.4064  }" />
+<xacro:property name="chassis_H" value="${0.1524   }" />
 <xacro:property name="bar_L" value="0.1" />
 <xacro:property name="bar_W" value="0.1" />
@@ -41,8 +41,8 @@
 <xacro:property name="ArmBase_x" value="0" />
 <xacro:property name="ArmBase_y" value="0" />
-<xacro:property name="ArmBase_z" value="0" />
+<xacro:property name="ArmBase_z" value="0.01" />
 <!-- Masses -->
-<xacro:property name="chassis_mass" value="600" />
+<xacro:property name="chassis_mass" value="100" />
 <xacro:property name="bar_mass" value="1" />
-<xacro:property name="wheels_mass" value="2" />
+<xacro:property name="wheels_mass" value="20" />
 </robot>
