Commit message: adding the arm controller

File: src/jaguar_pkg/parts/arm.xacro (robot description, xacro)
@@ -1,7 +1,8 @@
 <?xml version="1.0" ?>
 <robot xmlns:xacro="http://www.ros.org/wiki/xacro">
+<xacro:property name="joint_friction" value="5"/>
 <m_joint_1 name="${link_00_name}__${link_01_name}" type="revolute"
            axis_xyz="0 0 1"
-           damp="0.2" frict="50"
+           damp="0.2" frict="${joint_friction}"
            origin_rpy="0 0 0" origin_xyz="${0.13 * arm_scale_x }  ${0 * arm_scale_y } ${0.27 * arm_scale_z }"
            parent="${link_00_name}" child="${link_01_name}"
@@ -15,6 +16,7 @@
               meshfile="${the_meshfile}/Arm_Base_scaled.dae"
               meshscale="${arm_scale_x} ${arm_scale_y} ${arm_scale_z}" />
- <m_joint name="${link_01_name}__${link_06_name}" type="revolute"
+ <m_joint_1 name="${link_01_name}__${link_06_name}" type="revolute"
            axis_xyz="0 1 0"
+           damp="0.2" frict="${joint_friction}"
            origin_rpy="0 0.05 0" origin_xyz="${0.1 * arm_scale_x } ${0.039  * arm_scale_y } ${0.12 * arm_scale_z}"
            parent="${link_01_name}" child="${link_06_name}"
@@ -28,6 +30,7 @@
               meshfile="${the_meshfile}/Arm_1_scaled.dae"
               meshscale="${arm_scale_x} ${arm_scale_y} ${arm_scale_z}" />
-    <m_joint name="${link_06_name}__${link_07_name}" type="revolute"
+  <m_joint_1 name="${link_06_name}__${link_07_name}" type="revolute"
            axis_xyz="0 1 0"
+           damp="0.2" frict="${joint_friction}"
            origin_rpy="0 0 3.14" origin_xyz="${-0.46 * arm_scale_x } ${-0.1275 * arm_scale_y } ${0 * arm_scale_z }"
            parent="${link_06_name}" child="${link_07_name}"
@@ -41,6 +44,7 @@
               meshfile="${the_meshfile}/Arm_2_scaled.dae"
               meshscale="${arm_scale_x} ${arm_scale_y} ${arm_scale_z}" />
-  <m_joint name="${link_07_name}__${link_08_name}" type="revolute"
+  <m_joint_1 name="${link_07_name}__${link_08_name}" type="revolute"
            axis_xyz="0 1 0"
+           damp="0.2" frict="${joint_friction}"
            origin_rpy="0 0 0" origin_xyz="${-0.43 * arm_scale_x } ${-0.044 * arm_scale_y } ${0.14 * arm_scale_z }"
            parent="${link_07_name}" child="${link_08_name}"
@@ -54,6 +58,7 @@
               meshfile="${the_meshfile}/Arm_3_scaled.dae"
               meshscale="${arm_scale_x} ${arm_scale_y} ${arm_scale_z}" />
-  <m_joint name="${link_08_name}__${link_09_name}" type="revolute"
+  <m_joint_1 name="${link_08_name}__${link_09_name}" type="revolute"
            axis_xyz="1 0 0"
+           damp="0.2" frict="${joint_friction}"
            origin_rpy="0 -0.18 3.14" origin_xyz="${-0.08 * arm_scale_x } ${-0.0346 * arm_scale_y } ${0.014 * arm_scale_z }"
            parent="${link_08_name}" child="${link_09_name}"

File: src/jaguar_pkg/urdf/links_joints.xacro (robot description, xacro)
@@ -32,8 +32,8 @@
       <type>transmission_interface/SimpleTransmission</type>
       <joint name="${name}">
-        <hardwareInterface>hardware_interface/EffortJointInterface</hardwareInterface>
+        <hardwareInterface>hardware_interface/PositionJointInterface</hardwareInterface>
       </joint>
       <actuator name="motor_${name}">
-        <hardwareInterface>hardware_interface/EffortJointInterface</hardwareInterface>
+        <hardwareInterface>hardware_interface/PositionJointInterface</hardwareInterface>
         <mechanicalReduction>1</mechanicalReduction>
       </actuator>

Commit message: improving the collision tag

File: src/jaguar_pkg/parts/arm.xacro (robot description, xacro)
@@ -1,5 +1,7 @@
 <?xml version="1.0" ?>
 <robot xmlns:xacro="http://www.ros.org/wiki/xacro">
+ <!-- <xacro:include filename="$(find jaguar_pkg)/gazebo_plugins/arm.gazebo" /> -->
 <xacro:property name="joint_friction" value="5"/>
+<!-- base arm -->
 <m_joint_1 name="${link_00_name}__${link_01_name}" type="revolute"
            axis_xyz="0 0 1"
@@ -16,4 +18,5 @@
               meshfile="${the_meshfile}/Arm_Base_scaled.dae"
               meshscale="${arm_scale_x} ${arm_scale_y} ${arm_scale_z}" />
+<!-- arm 1 -->
  <m_joint_1 name="${link_01_name}__${link_06_name}" type="revolute"
            axis_xyz="0 1 0"
@@ -30,4 +33,5 @@
               meshfile="${the_meshfile}/Arm_1_scaled.dae"
               meshscale="${arm_scale_x} ${arm_scale_y} ${arm_scale_z}" />
+    <!-- arm 2 -->
   <m_joint_1 name="${link_06_name}__${link_07_name}" type="revolute"
            axis_xyz="0 1 0"
@@ -44,4 +48,5 @@
               meshfile="${the_meshfile}/Arm_2_scaled.dae"
               meshscale="${arm_scale_x} ${arm_scale_y} ${arm_scale_z}" />
+<!-- arm 3 -->
   <m_joint_1 name="${link_07_name}__${link_08_name}" type="revolute"
            axis_xyz="0 1 0"
@@ -49,5 +54,5 @@
            origin_rpy="0 0 0" origin_xyz="${-0.43 * arm_scale_x } ${-0.044 * arm_scale_y } ${0.14 * arm_scale_z }"
            parent="${link_07_name}" child="${link_08_name}"
-           limit_e="1000" limit_l="0" limit_u="0" limit_v="0" />
+           limit_e="1000" limit_l="-3.14" limit_u="3.14" limit_v="0.5" />
   <m_link_mesh name="${link_08_name}"
               origin_rpy="0 0 3.14" origin_xyz="0 0 0"
@@ -58,4 +63,5 @@
               meshfile="${the_meshfile}/Arm_3_scaled.dae"
               meshscale="${arm_scale_x} ${arm_scale_y} ${arm_scale_z}" />
+ <!-- gripper -->
   <m_joint_1 name="${link_08_name}__${link_09_name}" type="revolute"
            axis_xyz="1 0 0"

File: src/jaguar_pkg/parts/fins.xacro (robot description, xacro)
@@ -1,9 +1,10 @@
 <?xml version="1.0" ?>
 <robot xmlns:xacro="http://www.ros.org/wiki/xacro">
+ <!-- <xacro:include filename="$(find jaguar_pkg)/gazebo_plugins/fins.gazebo" /> -->
    <xacro:property name="_x" value="${chassis_L/2 - wheel_R}" />
 <!-- Front Left -->
   <m_joint name="${link_00_name}__${link_12_name}" type="continuous"
            axis_xyz="0 1 0"
-           origin_rpy="0 2.97 3.14" origin_xyz="${_x} ${ chassis_W/2 + wheel_L + fin_w + wheels_offset*3 }  ${wheel_R}"
+           origin_rpy="0 2.97 3.14" origin_xyz="${_x} ${ chassis_W/2 + wheel_L + fin_w + wheels_offset + fins_offset }  ${wheel_R}"
            parent="${link_00_name}" child="${link_12_name}"
            limit_e="1000" limit_l="-1.57" limit_u="1.57" limit_v="0.5" />
@@ -19,5 +20,5 @@
    <m_joint name="${link_00_name}__${link_13_name}" type="continuous"
            axis_xyz="0 1 0"
-           origin_rpy="0 0 0" origin_xyz="${- _x} ${ chassis_W/2 + wheel_L + fin_w + wheels_offset*3 }  ${wheel_R}"
+           origin_rpy="0 0 0" origin_xyz="${- _x} ${ chassis_W/2 + wheel_L + fin_w + wheels_offset + fins_offset }  ${wheel_R}"
            parent="${link_00_name}" child="${link_13_name}"
            limit_e="1000" limit_l="-1.57" limit_u="1.57" limit_v="0.5" />
@@ -33,5 +34,5 @@
    <m_joint name="${link_00_name}__${link_14_name}" type="continuous"
            axis_xyz="0 1 0"
-           origin_rpy="0 -0.17 3.14" origin_xyz="${_x} ${ -(chassis_W/2 + wheel_L + fin_w + wheels_offset*3) }  ${wheel_R}"
+           origin_rpy="0 -0.17 3.14" origin_xyz="${_x} ${ -(chassis_W/2 + wheel_L + fin_w + wheels_offset + fins_offset) }  ${wheel_R}"
            parent="${link_00_name}" child="${link_14_name}"
            limit_e="1000" limit_l="-1.57" limit_u="1.57" limit_v="0.5" />
@@ -47,5 +48,5 @@
   <m_joint name="${link_00_name}__${link_15_name}" type="continuous"
            axis_xyz="0 1 0"
-           origin_rpy="0 0 0" origin_xyz="${- _x} ${-(chassis_W/2 + wheel_L + fin_w + wheels_offset*3)}  ${wheel_R}"
+           origin_rpy="0 0 0" origin_xyz="${- _x} ${-(chassis_W/2 + wheel_L + fin_w + wheels_offset + fins_offset)}  ${wheel_R}"
            parent="${link_00_name}" child="${link_15_name}"
            limit_e="1000" limit_l="-1.57" limit_u="1.57" limit_v="0.5" />

File: src/jaguar_pkg/parts/velodyne.xacro (robot description, xacro)
@@ -11,4 +11,5 @@
   <link name="${link_tail}" >
     <visual>
+          <origin xyz="0 0 0"/>
       <geometry>
         <box size="${0.05 * scale_all} ${0.05 * scale_all} ${0.53 * scale_all}" />
@@ -17,5 +18,5 @@
     <collision>
       <geometry>
-        <box size="${0.5 * scale_all} ${0.5 * scale_all} ${0.1 * scale_all}" />
+        <box size="${0.05 * scale_all} ${0.05 * scale_all} ${0.53 * scale_all}" />
       </geometry>
     </collision>

File: src/jaguar_pkg/parts/wheels.xacro (robot description, xacro)
@@ -1,7 +1,8 @@
 <?xml version="1.0" ?>
-<robot xmlns:xacro="http://www.ros.org/wiki/xacro">
+<robot  name="jaguar" xmlns:xacro="http://www.ros.org/wiki/xacro">
 <!-- include gazebo plugins -->
  <xacro:include filename="$(find jaguar_pkg)/gazebo_plugins/wheels.gazebo" />
   <xacro:property name="_x" value="${chassis_L/2 - wheel_R}" /> <!-- 0.27 -->
+  <!-- left front wheel -->
   <m_joint name="${link_00_name}__${link_02_name}" type="continuous"
            axis_xyz="0 1 0"
@@ -9,5 +10,5 @@
            parent="${link_00_name}" child="${link_02_name}"
            limit_e="1000" limit_l="-3.14" limit_u="3.14" limit_v="0.5"  />
-  <m_link_mesh name="${link_02_name}"
+  <m_link_mesh_cylinder name="${link_02_name}"
               origin_rpy="0 0 0" origin_xyz="0 0 0"
               mass="${wheels_mass}"
@@ -15,6 +16,9 @@
               iyy="0.1" iyz="0"
               izz="0.1"
+              collision_origin_rpy="0 1.57079 1.57079"
+              collisionn_radius="${wheel_R}" collisionn_length="${wheel_L + wheel_L*.45 }"
               meshfile="${the_meshfile}/wheel.dae"
               meshscale="${wheel_scale_r} ${wheel_scale_l} ${wheel_scale_r}"/>
+<!-- right front wheel -->
     <m_joint name="${link_00_name}__${link_03_name}" type="continuous"
            axis_xyz="0 1 0"
@@ -22,12 +26,15 @@
            parent="${link_00_name}" child="${link_03_name}"
            limit_e="1000" limit_l="-3.14" limit_u="3.14" limit_v="0.5" />
-    <m_link_mesh name="${link_03_name}"
-                origin_rpy="0 0 0" origin_xyz="0 0 0"
-                mass="${wheels_mass}"
+    <m_link_mesh_cylinder name="${link_03_name}"
+              origin_rpy="0 0 0" origin_xyz="0 0 0"
+              mass="${wheels_mass}"
               ixx="0.1" ixy="0" ixz="0"
               iyy="0.1" iyz="0"
               izz="0.1"
-                meshfile="${the_meshfile}/wheel.dae"
-                meshscale="${wheel_scale_r} ${wheel_scale_l} ${wheel_scale_r}" />
+              collision_origin_rpy="0 1.57079 1.57079"
+              collisionn_radius="${wheel_R}" collisionn_length="${wheel_L + wheel_L*.45 }"
+              meshfile="${the_meshfile}/wheel.dae"
+              meshscale="${wheel_scale_r} ${wheel_scale_l} ${wheel_scale_r}" />
+<!-- right back wheel -->
     <m_joint name="${link_00_name}__${link_04_name}" type="continuous"
            axis_xyz="0 1 0"
@@ -35,5 +42,5 @@
            parent="${link_00_name}" child="${link_04_name}"
            limit_e="1000" limit_l="-3.14" limit_u="3.14" limit_v="0.5" />
-  <m_link_mesh name="${link_04_name}"
+  <m_link_mesh_cylinder name="${link_04_name}"
               origin_rpy="0 0 0" origin_xyz="0 0 0"
               mass="${wheels_mass}"
@@ -41,6 +48,9 @@
               iyy="0.1" iyz="0"
               izz="0.1"
+              collision_origin_rpy="0 1.57079 1.57079"
+              collisionn_radius="${wheel_R}" collisionn_length="${wheel_L + wheel_L*.45 }"
               meshfile="${the_meshfile}/wheel.dae"
               meshscale="${wheel_scale_r} ${wheel_scale_l} ${wheel_scale_r}" />
+<!-- left back wheel -->
       <m_joint name="${link_00_name}__${link_05_name}" type="continuous"
            axis_xyz="0 1 0"
@@ -48,5 +58,5 @@
            parent="${link_00_name}" child="${link_05_name}"
            limit_e="1000" limit_l="-3.14" limit_u="3.14" limit_v="0.5" />
-  <m_link_mesh name="${link_05_name}"
+  <m_link_mesh_cylinder name="${link_05_name}"
               origin_rpy="0 0 0" origin_xyz="0 0 0"
               mass="${wheels_mass}"
@@ -54,4 +64,6 @@
               iyy="0.1" iyz="0"
               izz="0.1"
+              collision_origin_rpy="0 1.57079 1.57079"
+              collisionn_radius="${wheel_R}" collisionn_length="${wheel_L + wheel_L*.45 }"
               meshfile="${the_meshfile}/wheel.dae"
               meshscale="${wheel_scale_r} ${wheel_scale_l} ${wheel_scale_r}" />

File: src/jaguar_pkg/urdf/jaguar.xacro (robot description, xacro)
@@ -5,5 +5,5 @@
   <!-- Begin - Include parts-->
    <!-- <xacro:include filename="$(find jaguar_pkg)/parts/tankWheel.xacro" />  -->
-  <xacro:include filename="$(find jaguar_pkg)/parts/fins.xacro" />
+  <!-- <xacro:include filename="$(find jaguar_pkg)/parts/fins.xacro" />   -->
   <xacro:include filename="$(find jaguar_pkg)/parts/wheels.xacro" />
   <xacro:include filename="$(find jaguar_pkg)/parts/arm.xacro" />
@@ -17,5 +17,5 @@
     <child link="${link_00_name}"/>
   </joint>
-  <m_link_mesh name="${link_00_name}"
+  <m_link_mesh_box name="${link_00_name}"
               origin_rpy="0 0 0" origin_xyz="0 0 ${wheel_R}"
               mass="${chassis_mass}"
@@ -23,5 +23,30 @@
               iyy="0.1" iyz="0"
               izz="0.1"
+              collisionn="${chassis_L} ${chassis_W} ${chassis_H}"
               meshfile="${the_meshfile}/jaguar_base.dae"
               meshscale="${chassis_scale_x} ${chassis_scale_y} ${chassis_scale_z}"/>
+  <!-- <joint name="${dummy_link}__${link_00_name}_1" type="fixed">
+    <parent link="${dummy_link}"/>
+    <child link="${link_00_name}_1"/>
+  </joint>
+  <link name="${link_00_name}_1" >
+    <visual>
+          <origin xyz="0 0 ${wheel_R}"/>
+      <geometry>
+        <box size="${chassis_L} ${chassis_W} ${chassis_H}" />
+      </geometry>
+    </visual>
+    <collision>
+      <geometry>
+        <box size="${chassis_L} ${chassis_W} ${chassis_H}" />
+      </geometry>
+    </collision>
+    <inertial>
+      <origin xyz="0 0 ${wheel_R}"/>
+      <mass value="${tail_mass}"/>
+      <inertia ixx="3.0" ixy="0.0" ixz="0.0"
+               iyy="3.0" iyz="0.0"
+               izz="3.0" />
+    </inertial>
+  </link> -->
 </robot>

File: src/jaguar_pkg/urdf/links_joints.xacro (robot description, xacro)
@@ -104,3 +104,47 @@
     </link>
   </xacro:macro>
+    <xacro:macro name="m_link_mesh_box" params="name collisionn origin_xyz origin_rpy meshfile meshscale mass ixx ixy ixz iyy iyz izz">
+      <link name="${name}">
+        <inertial>
+          <mass value="${mass}" />
+          <origin rpy="${origin_rpy}" xyz="${origin_xyz}" />
+          <inertia ixx="${ixx}" ixy="${ixy}" ixz="${ixz}" iyy="${iyy}" iyz="${iyz}" izz="${izz}" />
+        </inertial>
+        <collision>
+          <origin rpy="${origin_rpy}" xyz="${origin_xyz}" />
+          <geometry>
+            <box size="${collisionn}" />
+          </geometry>
+        </collision>
+        <visual>
+          <origin rpy="${origin_rpy}" xyz="${origin_xyz}" />
+          <geometry>
+            <mesh filename="${meshfile}" scale="${meshscale}"/>
+          </geometry>
+          <material name="light_black"/>
+        </visual>
+      </link>
+     </xacro:macro>
+    <xacro:macro name="m_link_mesh_cylinder" params="name collisionn_radius  collision_origin_rpy collisionn_length origin_xyz origin_rpy meshfile meshscale mass ixx ixy ixz iyy iyz izz">
+      <link name="${name}">
+        <inertial>
+          <mass value="${mass}" />
+          <origin rpy="${origin_rpy}" xyz="${origin_xyz}" />
+          <inertia ixx="${ixx}" ixy="${ixy}" ixz="${ixz}" iyy="${iyy}" iyz="${iyz}" izz="${izz}" />
+        </inertial>
+        <collision>
+          <origin rpy="${collision_origin_rpy}" xyz="${origin_xyz}" />
+          <geometry>
+            <cylinder radius="${collisionn_radius}" length="${collisionn_length}"/>
+          </geometry>
+        </collision>
+        <visual>
+          <origin rpy="${origin_rpy}" xyz="${origin_xyz}" />
+          <geometry>
+            <mesh filename="${meshfile}" scale="${meshscale}"/>
+          </geometry>
+          <material name="light_black"/>
+        </visual>
+      </link>
+    </xacro:macro>
 </robot>

File: src/jaguar_pkg/urdf/robot_parameters.xacro (robot description, xacro)
@@ -4,8 +4,8 @@
   <xacro:property name="link_00_name" value="chassis" />
   <xacro:property name="link_01_name" value="base_arm" />
-  <xacro:property name="link_02_name" value="wheel_front_left" />
-  <xacro:property name="link_03_name" value="wheel_front_right" />
-  <xacro:property name="link_04_name" value="wheel_back_right" />
-  <xacro:property name="link_05_name" value="wheel_back_left" />
+  <xacro:property name="link_02_name" value="wheel_left_front" />
+  <xacro:property name="link_03_name" value="wheel_right_front" />
+  <xacro:property name="link_04_name" value="wheel_right_back" />
+  <xacro:property name="link_05_name" value="wheel_left_back" />
   <xacro:property name="link_06_name" value="arm_1" />
   <xacro:property name="link_07_name" value="arm_2" />
@@ -36,7 +36,7 @@
   <xacro:property name="lidar_scale" value="${0.001 * scale_all}" />
   <xacro:property name="off_The_Ground" value="0.01" />
-  <xacro:property name="chassis_L" value="${0.6858  *  chassis_scale_x }" />
-  <xacro:property name="chassis_W" value="${0.4064  *  chassis_scale_y }" />
-  <xacro:property name="chassis_H" value="${0.1524  *  chassis_scale_z }" />
+  <xacro:property name="chassis_L" value="${ 0.6858  *  chassis_scale_x }" />
+  <xacro:property name="chassis_W" value="${ 0.4064  *  chassis_scale_y }" />
+  <xacro:property name="chassis_H" value="${ 0.1524  *  chassis_scale_z }" />
   <xacro:property name="wheel_R" value="${0.0545 * wheel_scale_r}" />
   <xacro:property name="wheel_L" value="${0.0109 * wheel_scale_l}" />
@@ -44,12 +44,13 @@
   <!-- off set the wheel from the chassis -->
   <xacro:property name="wheels_offset" value="0.001" />
+  <xacro:property name="fins_offset" value="0.001" />
   <xacro:property name="lidar_x" value="0" />
  <xacro:property name="lidar_y" value="${ - chassis_W/2 + (0.04 * scale_all) }"/>
-  <xacro:property name="lidar_z" value="${0.02 * scale_all}" />
+  <xacro:property name="lidar_z" value="${0.03 * scale_all}" />
   <!-- Masses -->
-  <xacro:property name="chassis_mass" value="${ 100 * scale_all }" />
-  <xacro:property name="wheels_mass" value="${ 10 * scale_all }" />
-  <xacro:property name="fins_mass" value="${ 10 * scale_all }" />
-  <xacro:property name="arm_mass" value="${ 5 * scale_all }" />
-  <xacro:property name="tail_mass" value="${ 10 * scale_all }" />
+  <xacro:property name="chassis_mass" value="${ 100  }" />
+  <xacro:property name="wheels_mass" value="${ 1 * scale_all }" />
+  <xacro:property name="fins_mass" value="${ 1 * scale_all }" />
+  <xacro:property name="arm_mass" value="${ 1 * scale_all }" />
+  <xacro:property name="tail_mass" value="${ 1 * scale_all }" />
 </robot>
