Commit message: backup

File: src/jaguar_pkg/parts/velodyne.xacro (robot description, xacro)
@@ -29,5 +29,5 @@
     </inertial>
   </link>
- <VLP-16 parent="${link_tail}" name="velodyne" topic="/velodyne_points" hz="10" samples="440" gpu="${gpu}" scaleModel="${scale_all}">
+  <VLP-16 parent="${link_tail}" name="velodyne" topic="/velodyne_points" hz="10" samples="440" gpu="${gpu}" scaleModel="${scale_all}">
     <origin xyz="0 0 ${0.27 * scale_all}" rpy="0 0 0" />
   </VLP-16>

File: src/jaguar_pkg/parts/velodyne_des.xacro (robot description, xacro)
@@ -27,7 +27,7 @@
       </visual>
       <collision>
-        <origin rpy="0 0 0" xyz="0 0 0.03585"/>
+        <origin rpy="0 0 0" xyz="0 0 ${0.03585 * scaleModel}"/>
         <geometry>
-          <cylinder radius="0.0516" length="0.0717"/>
+          <cylinder radius="${0.0516 * scaleModel}" length="${0.0717 * scaleModel}"/>
         </geometry>
       </collision>

File: src/jaguar_pkg/urdf/jaguar.xacro (robot description, xacro)
@@ -1,9 +1,10 @@
 <?xml version="1.0" ?>
 <robot name="jaguar" xmlns:xacro="http://www.ros.org/wiki/xacro">
-  <xacro:include filename="$(find jaguar_pkg)/urdf/robot_parameters.xacro" />
-  <xacro:include filename="$(find jaguar_pkg)/urdf/links_joints.xacro" />
+  <xacro:include filename="$(find jaguar_pkg)/lib/robot_parameters.xacro" />
+  <xacro:include filename="$(find jaguar_pkg)/lib/links_joints.xacro" />
   <!-- Begin - Include parts-->
-   <!-- <xacro:include filename="$(find jaguar_pkg)/parts/tankWheel.xacro" />  -->
-  <!-- <xacro:include filename="$(find jaguar_pkg)/parts/fins.xacro" />   -->
+  <!-- <xacro:include filename="$(find jaguar_pkg)/parts/tankWheel.xacro" />   -->
+  <!-- <xacro:include filename="$(find jaguar_pkg)/parts/fins.xacro" />    -->
+  <xacro:include filename="$(find jaguar_pkg)/parts/_d435.urdf.xacro" />
   <xacro:include filename="$(find jaguar_pkg)/parts/wheels.xacro" />
   <xacro:include filename="$(find jaguar_pkg)/parts/arm.xacro" />
